Commit message: complete joint-space shadow planner + task space robot

File: gibson2/assets/models/grippers/cube_gripper/gripper.urdf (robot description, URDF)
Before this commit: robot cube_gripper, 8 links, 7 joints
Joints:
- joint txj: limit lower=-1.0 upper=1.0 -> lower=-2.0 upper=2.0
- joint tyj: limit lower=-1.0 upper=1.0 -> lower=-2.0 upper=2.0
