Commit message: simple tool env assets

File: gibson2/assets/models/grippers/basic_gripper/gripper.urdf (robot description, URDF)
Before this commit: robot basic_gripper, 6 links, 5 joints
Links:
- link eef_link: geometry 

File: gibson2/assets/models/grippers/basic_gripper/gripper_plannable.urdf (robot description, URDF)
Before this commit: robot basic_gripper, 12 links, 11 joints
Links:
- link eef_link: geometry 
