Commit message: add support for wrist camera on fetch robot

File: gibson2/data/assets/models/fetch/fetch_gripper.urdf (robot description, URDF)
Before this commit: robot fetch, 26 links, 25 joints
Links:
- added link eyes_wrist, mass 0.001
Joints:
- added joint wrist_eye_joint: type fixed, parent gripper_link, child eyes_wrist, origin xyz=-0.16 0 -0.1 rpy=3.141592654 -0.2 0

File: gibson2/data/assets/models/fetch/fetch_gripper_vis.urdf (robot description, URDF)
Before this commit: robot fetch, 26 links, 25 joints
Links:
- added link eyes_wrist, mass 0.001
Joints:
- added joint wrist_eye_joint: type fixed, parent gripper_link, child eyes_wrist, origin xyz=-0.16 0 -0.1 rpy=3.141592654 -0.2 0
