Commit message: remove wrist camera from vis version of fetch robot

File: gibson2/data/assets/models/fetch/fetch_gripper_vis.urdf (robot description, URDF)
Before this commit: robot fetch, 27 links, 26 joints
Links:
- removed link eyes_wrist
Joints:
- removed joint wrist_eye_joint

Commit message: add trash to env, add sampling functionality to ycb objects, modify cube object to work with sampling API, increase fetch robot gripper friction

File: gibson2/data/assets/models/fetch/fetch_gripper_vis.urdf (robot description, URDF)
Before this commit: robot fetch, 26 links, 25 joints
Links:
- link gripper_link: geometry collision mesh filename=meshes/gripper_link.obj; visual box size=0.004 0.004 0.4
