Commit message: fix sim bugs for waking up objects, tune ik controller

File: gibson2/data/ig_dataset/scenes/Pomaria_1_int/urdf/Pomaria_1_int_custom_kitchen.urdf (robot description, URDF)
Before this commit: robot igibson_scene, 72 links, 71 joints
Links:
- removed link chair_1
- removed link chair_2
- removed link chair_7
- removed link chair_8
- removed link coffee_table_3
- removed link coffee_table_4
- removed link desk_76
- removed link plant_5
- removed link table_6
Joints:
- removed joint j_chair_1
- removed joint j_chair_2
- removed joint j_chair_7
- removed joint j_chair_8
- removed joint j_coffee_table_3
- removed joint j_coffee_table_4
- removed joint j_desk_76
- removed joint j_plant_5
- removed joint j_table_6
- joint j_bottom_cabinet_26: origin xyz=-2.705000 -2.625000 0.450000 rpy=0 0 -3.141593 -> xyz=-2.505000 -2.625000 0.450000 rpy=0 0 -3.141593
- joint j_bottom_cabinet_no_top_38: origin xyz=-4.115000 -2.639000 0.450000 rpy=0 0 -3.141593 -> xyz=-3.915000 -2.639000 0.450000 rpy=0 0 -3.141593
- joint j_cooktop_64: origin xyz=-3.580000 -2.630000 0.940000 rpy=0 0 -3.141593 -> xyz=-3.180000 -2.630000 0.940000 rpy=0 0 -3.141593
- joint j_counter_41: origin xyz=-4.140000 -2.650000 0.910500 rpy=0 0 0.000000 -> xyz=-3.940000 -2.650000 0.910500 rpy=0 0 0.000000
- joint j_oven_46: origin xyz=-3.580000 -2.630000 0.450000 rpy=0 0 -3.141593 -> xyz=-3.180000 -2.630000 0.450000 rpy=0 0 -3.141593
