Commit message: add three location setup

File: gibson2/data/ig_dataset/scenes/Pomaria_1_int/urdf/Pomaria_1_int_custom_multilocation3.urdf (robot description, URDF)
Before this commit: robot igibson_scene, 81 links, 80 joints
Links:
- added link dishwasher_78
Joints:
- added joint j_dishwasher_78: type fixed, parent world, child dishwasher_78, origin xyz=-13. 0.0 0.450000 rpy=0 0 1.5708
- joint j_cabinet_77: origin xyz=-11.15 -2.2 0.45 rpy=0 0 3.141593 -> xyz=-9.15 -2.2 0.45 rpy=0 0 4.1888
- joint j_desk_76: origin xyz=-11.15 2.2 0.45 rpy=0 0 0 -> xyz=-9.15 2.2 0.45 rpy=0 0 -0.5236

Commit message: fix cabinet2 ori in 3 location setup

File: gibson2/data/ig_dataset/scenes/Pomaria_1_int/urdf/Pomaria_1_int_custom_multilocation3.urdf (robot description, URDF)
Before this commit: robot igibson_scene, 82 links, 81 joints
Joints:
- joint j_cabinet_77: origin xyz=-9.15 -2.2 0.45 rpy=0 0 4.1888 -> xyz=-9.15 -2.2 0.45 rpy=0 0 -2.6180
