Commit message: tune semantic organize and fetch env, fill in table cleanup urdf, fix reset bugs with fetch robot

File: gibson2/data/ig_dataset/scenes/Pomaria_1_int/urdf/Pomaria_1_int_custom_kitchen_cleanup_full.urdf (robot description, URDF)
Before this commit: robot igibson_scene, 7 links, 6 joints
Links:
- added link bottom_cabinet_26
- added link bottom_cabinet_no_top_29
- added link bottom_cabinet_no_top_30
- added link bottom_cabinet_no_top_32
- added link bottom_cabinet_no_top_35
- added link bottom_cabinet_no_top_38
- added link bottom_cabinet_no_top_39
- added link carpet_13
- added link carpet_34
- added link counter_31
- added link counter_33
- added link counter_40
- added link counter_41
- added link fridge_20
- added link microwave_23
- added link oven_21
- added link oven_22
- added link oven_46
- added link picture_17
- added link picture_18
- added link picture_19
- added link picture_28
- added link shelf_14
- added link shelf_15
- added link shelf_16
- added link sink_37
- added link table_0
- added link top_cabinet_24
- added link top_cabinet_25
- added link top_cabinet_27
- added link top_cabinet_42
- added link top_cabinet_43
Joints:
- added joint j_bottom_cabinet_26: type fixed, parent world, child bottom_cabinet_26, origin xyz=-4.405000 -1.185000 0.450000 rpy=0 0 -4.708644
- added joint j_bottom_cabinet_no_top_29: type fixed, parent world, child bottom_cabinet_no_top_29, origin xyz=-0.595000 0.625000 0.450000 rpy=0 0 0.000000
- added joint j_bottom_cabinet_no_top_30: type fixed, parent world, child bottom_cabinet_no_top_30, origin xyz=0.145000 0.625000 0.450000 rpy=0 0 0.000000
- added joint j_bottom_cabinet_no_top_32: type fixed, parent world, child bottom_cabinet_no_top_32, origin xyz=0.753266 -0.126519 0.450000 rpy=0 0 -1.569348
- added joint j_bottom_cabinet_no_top_35: type fixed, parent world, child bottom_cabinet_no_top_35, origin xyz=-4.505000 -1.815000 0.450000 rpy=0 0 -4.708644
- added joint j_bottom_cabinet_no_top_38: type fixed, parent world, child bottom_cabinet_no_top_38, origin xyz=-3.915000 -2.639000 0.450000 rpy=0 0 -3.141593
- added joint j_bottom_cabinet_no_top_39: type fixed, parent world, child bottom_cabinet_no_top_39, origin xyz=-4.507060 -2.217114 0.450000 rpy=0 0 -4.707637
- added joint j_carpet_13: type fixed, parent world, child carpet_13, origin xyz=-6.684743 -0.871725 0.000500 rpy=0 0 -1.555760
- added joint j_carpet_34: type fixed, parent world, child carpet_34, origin xyz=-0.497374 -1.683206 0.000500 rpy=0 0 -1.554614
- added joint j_counter_31: type fixed, parent world, child counter_31, origin xyz=0.035000 0.650000 0.910500 rpy=0 0 0.000000
- added joint j_counter_33: type fixed, parent world, child counter_33, origin xyz=0.780000 -0.100000 0.910500 rpy=0 0 0.000000
- added joint j_counter_40: type fixed, parent world, child counter_40, origin xyz=-4.520000 -1.925000 0.910500 rpy=0 0 -3.141593
- added joint j_counter_41: type fixed, parent world, child counter_41, origin xyz=-3.940000 -2.650000 0.910500 rpy=0 0 0.000000
- added joint j_fridge_20: type fixed, parent world, child fridge_20, origin xyz=-2.565000 0.550000 0.925000 rpy=0 0 0.000000
- added joint j_microwave_23: type fixed, parent world, child microwave_23, origin xyz=-4.350000 0.550000 1.700050 rpy=0 0 0.000000
- added joint j_oven_21: type fixed, parent world, child oven_21, origin xyz=-4.350000 0.550000 1.085050 rpy=0 0 0.000000
- added joint j_oven_22: type fixed, parent world, child oven_22, origin xyz=-4.350000 0.550000 0.360000 rpy=0 0 0.000000
- added joint j_oven_46: type fixed, parent world, child oven_46, origin xyz=-3.180000 -2.630000 0.450000 rpy=0 0 -3.141593
- added joint j_picture_17: type fixed, parent world, child picture_17, origin xyz=-12.870000 -1.870000 1.650000 rpy=0 0 1.570796
- added joint j_picture_18: type fixed, parent world, child picture_18, origin xyz=-12.890000 1.960000 1.650000 rpy=0 0 1.570796
- added joint j_picture_19: type fixed, parent world, child picture_19, origin xyz=-9.950000 2.985000 1.700000 rpy=0 0 0.000000
- added joint j_picture_28: type fixed, parent world, child picture_28, origin xyz=0.999546 0.075000 1.780000 rpy=0 0 -1.571645
- added joint j_shelf_14: type fixed, parent world, child shelf_14, origin xyz=-5.158734 -1.987750 1.100000 rpy=0 0 -1.574043
- added joint j_shelf_15: type fixed, parent world, child shelf_15, origin xyz=-12.628504 -1.902279 0.250000 rpy=0 0 1.568601
- added joint j_shelf_16: type fixed, parent world, child shelf_16, origin xyz=-12.638504 1.935683 0.250000 rpy=0 0 1.568601
- added joint j_sink_37: type fixed, parent world, child sink_37, origin xyz=-3.455000 0.630000 0.450000 rpy=0 0 0.000
- added joint j_table_0: type floating, parent world, child table_0, origin xyz=-8.250000 -2.590000 0.200000 rpy=0 0 -3.141593
- added joint j_top_cabinet_24: type fixed, parent world, child top_cabinet_24, origin xyz=-2.560000 0.560000 2.125050 rpy=0 0 0.000000
- added joint j_top_cabinet_25: type fixed, parent world, child top_cabinet_25, origin xyz=-4.345000 0.555000 2.175050 rpy=0 0 0.000000
- added joint j_top_cabinet_27: type fixed, parent world, child top_cabinet_27, origin xyz=-3.465000 0.630000 1.900000 rpy=0 0 0.000000
- added joint j_top_cabinet_42: type fixed, parent world, child top_cabinet_42, origin xyz=-4.655000 -1.395000 1.900000 rpy=0 0 1.570796
- added joint j_top_cabinet_43: type fixed, parent world, child top_cabinet_43, origin xyz=-4.645000 -2.445000 1.900000 rpy=0 0 1.570796
