Commit message: update oven location in pomaria generalize env

File: gibson2/data/ig_dataset/scenes/Pomaria_1_int/urdf/Pomaria_1_int_custom_kitchen_cleanup_full_generalize.urdf (robot description, URDF)
Before this commit: robot igibson_scene, 39 links, 38 joints
Joints:
- joint j_oven_46: origin xyz=-3.455000 0.630000 0.450000 rpy=0 0 0 -> xyz=-3.455000 0.550000 0.360000 rpy=0 0 0

Commit message: swap cabinet and dishwasher locations in generalize env

File: gibson2/data/ig_dataset/scenes/Pomaria_1_int/urdf/Pomaria_1_int_custom_kitchen_cleanup_full_generalize.urdf (robot description, URDF)
Before this commit: robot igibson_scene, 39 links, 38 joints
Joints:
- joint j_bottom_cabinet_26: origin xyz=-4.405000 -1.185000 0.450000 rpy=0 0 -4.708644 -> xyz=-2.505000 -2.625000 0.450000 rpy=0 0 -3.141593
- joint j_dishwasher_36: origin xyz=-2.505000 -2.625000 0.450000 rpy=0 0 -3.141593 -> xyz=-4.405000 -1.185000 0.450000 rpy=0 0 -4.708644

Commit message: tune bottom cabinet location in generalize env

File: gibson2/data/ig_dataset/scenes/Pomaria_1_int/urdf/Pomaria_1_int_custom_kitchen_cleanup_full_generalize.urdf (robot description, URDF)
Before this commit: robot igibson_scene, 39 links, 38 joints
Joints:
- joint j_bottom_cabinet_26: origin xyz=-2.505000 -2.625000 0.450000 rpy=0 0 -3.141593 -> xyz=-2.495000 -2.625000 0.450000 rpy=0 0 -3.141593
