Commit message: add extra handle to dishwasher, tune kitchen cleanup env, add cooldown to vertical head tilt heuristic for fetch

File: gibson2/data/ig_dataset/objects/dishwasher/12349_handle/12349_handle.urdf (robot description, URDF)
Before this commit: robot 12349, 4 links, 3 joints
Links:
- link link_1: geometry collision box size=0.30 0.01 0.025; collision mesh filename=shape/collision/link_1_cm.obj

File: gibson2/data/ig_dataset/scenes/Pomaria_1_int/urdf/Pomaria_1_int_custom_kitchen_cleanup.urdf (robot description, URDF)
Before this commit: robot igibson_scene, 7 links, 6 joints
Joints:
- joint j_table_76: origin xyz=-2.5 -1.3 0.395 rpy=0 0 0.000000 -> xyz=-2.0 -1.3 0.395 rpy=0 0 0.000000

File: gibson2/data/ig_dataset/scenes/Pomaria_1_int/urdf/Pomaria_1_int_custom_kitchen_cleanup_easy.urdf (robot description, URDF)
Before this commit: robot igibson_scene, 7 links, 6 joints
Joints:
- joint j_table_76: origin xyz=-2.5 -1.3 0.395 rpy=0 0 0.000000 -> xyz=-2.0 -1.3 0.395 rpy=0 0 0.000000
