Commit message: open joint in cabinet a little more

File: gibson2/data/ig_dataset/objects/bottom_cabinet/49140/49140.urdf (robot description, URDF)
Before this commit: robot 49140, 5 links, 4 joints
Joints:
- joint joint_3: limit lower=0.035 upper=1.0 -> lower=0.045 upper=1.0
- joint joint_4: limit lower=0.03 upper=1.0 -> lower=0.04 upper=1.0

Commit message: fix scaling bug for ycb objs, update object metadata, add functionality to randomize scene object poses

File: gibson2/data/ig_dataset/objects/bottom_cabinet/49140/49140.urdf (robot description, URDF)
Before this commit: robot 49140, 5 links, 4 joints
Joints:
- joint joint_3: limit lower=0.045 upper=1.0 -> lower=0.035 upper=1.0
- joint joint_4: limit lower=0.04 upper=1.0 -> lower=0.03 upper=1.0

File: gibson2/data/ig_dataset/scenes/Pomaria_1_int/urdf/Pomaria_1_int_custom_kitchen_cleanup_full.urdf (robot description, URDF)
Before this commit: robot igibson_scene, 39 links, 38 joints
Joints:
- joint j_table_76: origin xyz=-2.05000 -1.1000 0.395 rpy=0 0 0.000000 -> xyz=-2.05000 -0.9000 0.395 rpy=0 0 0.000000
- joint j_trash_can_77: origin xyz=-1.855000 -2.75000 0.400000 rpy=0 0 1.570796 -> xyz=-1.455000 -3.05000 0.400000 rpy=0 0 1.570796
