Commit message: [Visual Disease]
- Change dirty sampling to be solely on top, and clean threshold to be 0
- Add seed generation and task sequence generation files
- Add some task-related data
- Fix various bugs

File: igibson/examples/vr/visual_disease_demo_mtls/butter/butter_000.urdf (robot description, URDF)
Before this commit: robot butter_000, 1 links, 0 joints
Links:
- link base_link: mass 1.0 -> 3.0
