Commit message: [Visual Disease]
- Fix bugs in demo materials
- Add metadata and task specific data to ig logging
- Made simple task room smaller
- Fixed randomization bug in wipe

File: igibson/examples/vr/visual_disease_demo_mtls/basket/rectangle_basket.urdf (robot description, URDF)
Before this commit: robot e3bae8da192ab3d4a17ae19fa77775ff, 1 links, 0 joints
Links:
- link base_link: mass 1.0562898801609841 -> 100.0562898801609841; geometry collision mesh filename=shape/collision/e3bae8da192ab3d4a17ae19fa77775ff_cm.obj scale=1 0.8 0.4; visual mesh filename=shape/visual/e3bae8da192ab3d4a17ae19fa77775ff_m1_vm.encrypt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 scale=1 0.8 0.4

File: igibson/examples/vr/visual_disease_demo_mtls/basket/square_basket.urdf (robot description, URDF)
Before this commit: robot e3bae8da192ab3d4a17ae19fa77775ff, 1 links, 0 joints
Links:
- link base_link: mass 1.0562898801609841 -> 100.0562898801609841; geometry collision mesh filename=shape/collision/e3bae8da192ab3d4a17ae19fa77775ff_cm.obj scale=0.6 0.8 0.4; visual mesh filename=shape/visual/e3bae8da192ab3d4a17ae19fa77775ff_m1_vm.encrypt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 scale=0.6 0.8 0.4

File: igibson/examples/vr/visual_disease_demo_mtls/cube/square_cube.urdf (robot description, URDF)
Before this commit: robot butter_000, 1 links, 0 joints
Links:
- link base_link: geometry collision mesh filename=shape/collision/butter_000_cm.obj scale=0.05 0.0275 0.05; visual mesh filename=shape/visual/butter_package.encrypted.obj scale=0.05 0.0275 0.05

File: igibson/examples/vr/visual_disease_demo_mtls/plane/white_plane.urdf (robot description, URDF)
Before this commit: robot plane, 1 links, 0 joints
Links:
- link planeLink: geometry collision box size=30 30 1; visual mesh filename=plane.obj scale=1 1 1
