Commit message: [Visual Disease]
- Fix some bugs in vi rendering
- Clean up code

File: igibson/examples/vr/visual_disease_demo_mtls/plane/floor.urdf (robot description, URDF)
Before this commit: robot plane, 1 links, 0 joints
Links:
- link planeLink: geometry collision box size=100 100 0.01; visual mesh filename=floor.obj scale=1 1 1
